File: hardware/electronic/wordclock_v1_9.sch (EAGLE design)
At the start: 29 parts, among them IC3* REG1117, Q1* BS170

Commit message: Fix
Fix:
- ESP CH_PD pin pull up #21
- Wire RX/TX #20
- Fix main PCB label #10
Parts:
- removed EEPROM*: AT24CP, atmel:AT24CP
- removed I2C*: (no value), con-amp:MTA05-100
- removed JP3: (no value), PINHD8:90:PINHD-2X3
- removed JP4: (no value), PINHD8:90:PINHD-1X6
- removed R2*: 4k7, rcl:R-EU_0207/10
- removed R5*: 10k, rcl:R-EU_0207/10
- added D1: 1N4148, diode:1N4148DO35-10
- added I2C: (no value), con-amp:MTA05-100
- added R5, R8: 10k, rcl:R-EU_0207/10
- added R7: 4k7, rcl:R-EU_0207/10
- added RTC: (no value), PINHD8:90:PINHD-1X6
- added SET: (no value), pinhead:PINHD-1X2
- LED: device con-amp_3:MTA03-156 -> con-amp:MTA03-156
- renumbered C2* to C2, C3* to C3, ESP8266* to ESP8266, IC3* to IC3, Q1* to Q1, R3* to R3, R4* to R4, R6* to R6, R7* to R2, SENSOR* to SENSOR
Connections:
- removed net N$10: JP1.14, JP3.6, PCB2.RX0
- removed net TX: JP3.3, Q1.D, R5*.2
- new net N$1: ESP8266.CH_PD, R8.1
- new net N$12: D1.C, JP2.4, PCB2.5V
- net 3V3: now also I2C.2; no longer I2C*.2
- net GND: now also I2C.3, RTC.6, SET.2; no longer EEPROM*.A0, EEPROM*.A1, EEPROM*.A2, EEPROM*.GND, EEPROM*.WP, ESP8266.CH_PD, I2C*.3, JP3.2, JP4.6
- net N$11: now also Q1.D, R5.2; no longer JP3.4
- net RX: now also JP1.14, PCB2.RX0; no longer JP3.5
- net SCL: now also I2C.4, R2.1, RTC.3; no longer EEPROM*.SCL, I2C*.4, JP4.3, R2*.1
- net SDA: now also I2C.5, R7.1, RTC.4; no longer EEPROM*.SDA, I2C*.5, JP4.4, R2.1
- net SET: now also SET.1; no longer JP3.1
- net VCC: now also D1.A, I2C.1, R5.1, R7.2, R8.2, RTC.5; no longer EEPROM*.VCC, I2C*.1, JP2.4, JP4.5, PCB2.5V, R2*.2, R5*.1
Other:
- note removed: "DO"
- note removed: "SET"
